File: Schematics/IOTv1.kicad_pcb (KiCad board)
At the start: 2 copper layers, 29 x 26 mm, 14 parts, among them IC1 TPS7A2633DRVR, J1 USB_SMD_105450-0101, J2 Conn_01x04

Commit message: Add files via upload
Parts:
- removed Cin2, Cin3, Cin4, Cin5: 2.2uF, Capacitor_SMD:C_0402_1005Metric
- removed Rpg1, Rpg2, Rpg3: R_Small, Resistor_SMD:R_0402_1005Metric
- added C1: 10U, Capacitor_SMD:C_0402_1005Metric, F.Cu at (313.3, 70.7)
- added C10: 2.2uF, Capacitor_SMD:C_0402_1005Metric, B.Cu at (405.4, 82.4)
- added C11: 1uf, Capacitor_SMD:C_0402_1005Metric, F.Cu at (316.7, 81.8)
- added C12: 1uf, Capacitor_SMD:C_0402_1005Metric, F.Cu at (298.9, 94.8)
- added C13: 1uf, Capacitor_SMD:C_0402_1005Metric, F.Cu at (308.5, 92.3)
- added C14: 1uf, Capacitor_SMD:C_0402_1005Metric, F.Cu at (298.9, 96.8)
- added C15: 2.2uF, Capacitor_SMD:C_0402_1005Metric, B.Cu at (385.0, 89.6)
- added C16: 0.1U, Capacitor_SMD:C_0402_1005Metric, F.Cu at (313.3, 66.7)
- added C17: 1U, Capacitor_SMD:C_0402_1005Metric, F.Cu at (316.5, 62.3)
- added C18: 1U, Capacitor_SMD:C_0402_1005Metric, F.Cu at (313.6, 64.7)
- added C19: 10U, Capacitor_SMD:C_0402_1005Metric, F.Cu at (318.9, 60.3)
- added C2: 1U, Capacitor_SMD:C_0402_1005Metric, F.Cu at (310.4, 72.4)
- added C20: 2.2uF, Capacitor_SMD:C_0402_1005Metric, B.Cu at (386.4, 89.6)
- added C21: 10U, Capacitor_SMD:C_0402_1005Metric, F.Cu at (405.6, 116.3)
- added C22: 10U, Capacitor_SMD:C_0402_1005Metric, F.Cu at (408.5, 116.3)
- added C23: 1U, Capacitor_SMD:C_0402_1005Metric, F.Cu at (154.4, 82.5)
- added C24: 1U, Capacitor_SMD:C_0402_1005Metric, F.Cu at (154.4, 83.6)
- added C25: 1U, Capacitor_SMD:C_0402_1005Metric, F.Cu at (156.5, 80.4)
- added C26: 1U, Capacitor_SMD:C_0402_1005Metric, F.Cu at (153.8, 79.9)
- added C27: 1U, Capacitor_SMD:C_0402_1005Metric, F.Cu at (156.8, 78.3)
- added C28: 1U, Capacitor_SMD:C_0402_1005Metric, F.Cu at (159.7, 79.8)
- added C29: 1uf, Capacitor_SMD:C_0402_1005Metric, B.Cu at (157.1, 85.2)
- added C3: 1U, Capacitor_SMD:C_0402_1005Metric, F.Cu at (316.5, 66.3)
- added C30: 1uf, Capacitor_SMD:C_0402_1005Metric, B.Cu at (157.3, 90.1)
- added C31: 1U, Capacitor_SMD:C_0402_1005Metric, F.Cu at (155.4, 78.3)
- added C32: 1U, Capacitor_SMD:C_0402_1005Metric, F.Cu at (158.2, 79.4)
- added C33: 1U, Capacitor_SMD:C_0402_1005Metric, F.Cu at (158.7, 77.8)
- added C34: 1U, Capacitor_SMD:C_0402_1005Metric, F.Cu at (153.8, 76.8)
- added C35: 1uf, Capacitor_SMD:C_0402_1005Metric, F.Cu at (153.8, 85.3)
- added C36: 1N, Capacitor_SMD:C_0402_1005Metric, F.Cu at (154.9, 74.5)
- added C37: 1N, Capacitor_SMD:C_0402_1005Metric, F.Cu at (158.8, 74.5)
- added C38: 1N, Capacitor_SMD:C_0402_1005Metric, F.Cu at (157.3, 72.9)
- added C39: 470N, Capacitor_SMD:C_0402_1005Metric, F.Cu at (155.1, 92.1)
- added C4: 0.1U, Capacitor_SMD:C_0402_1005Metric, F.Cu at (319.5, 64.3)
- added C40: 1N, Capacitor_SMD:C_0402_1005Metric, F.Cu at (155.8, 71.3)
- added C41: 1U, Capacitor_SMD:C_0402_1005Metric, F.Cu at (158.3, 91.3)
- added C42: 1N, Capacitor_SMD:C_0402_1005Metric, F.Cu at (158.0, 71.3)
- added C43: 0.1U, Capacitor_SMD:C_0402_1005Metric, F.Cu at (310.4, 70.4)
- added C44: 270P, Capacitor_SMD:C_0402_1005Metric, F.Cu at (316.0, 60.3)
- added C45: 270P, Capacitor_SMD:C_0402_1005Metric, F.Cu at (318.9, 58.3)
- added C46: 0.1U, Capacitor_SMD:C_0402_1005Metric, F.Cu at (310.4, 68.4)
- added C47: 0.1U, Capacitor_SMD:C_0402_1005Metric, F.Cu at (310.7, 62.7)
- added C48: 1U, Capacitor_SMD:C_0402_1005Metric, F.Cu at (294.8, 73.6)
- added C49: 1U, Capacitor_SMD:C_0402_1005Metric, F.Cu at (316.0, 58.3)
- added C5: 100P, Capacitor_SMD:C_0402_1005Metric, F.Cu at (316.5, 64.3)
- added C50: 270P, Capacitor_SMD:C_0402_1005Metric, F.Cu at (319.2, 68.2)
- added C51: 0.1U, Capacitor_SMD:C_0402_1005Metric, F.Cu at (316.2, 70.2)
- added C52: 0.1U, Capacitor_SMD:C_0402_1005Metric, F.Cu at (316.2, 68.2)
- added C53: 0.1U, Capacitor_SMD:C_0402_1005Metric, F.Cu at (319.5, 62.3)
- added C54: 10U, Capacitor_SMD:C_0402_1005Metric, F.Cu at (313.3, 68.7)
- added C55: 4.7U, Capacitor_SMD:C_0402_1005Metric, B.Cu at (387.8, 89.6)
- added C6: 1U, Capacitor_SMD:C_0402_1005Metric, F.Cu at (319.5, 66.3)
- added C7: 2.2uF, Capacitor_SMD:C_0402_1005Metric, B.Cu at (428.6, 69.8)
- added C8: 0.1U, Capacitor_SMD:C_0402_1005Metric, F.Cu at (313.3, 72.7)
- added C9: 2.2uF, Capacitor_SMD:C_0402_1005Metric, B.Cu at (407.2, 82.4)
- added D3: PMEG1030EJ, Diode_SMD:D_SOD-323F, B.Cu at (384.6, 87.6)
- added D4: LED, LED_SMD:LED_0402_1005Metric, B.Cu at (391.4, 84.8)
- added D5: LED, LED_SMD:LED_0402_1005Metric, B.Cu at (391.4, 82.4)
- added D6: LED, LED_SMD:LED_0402_1005Metric, B.Cu at (391.4, 87.8)
- added D7: PMEG1030EJ, Diode_SMD:D_SOD-323F, B.Cu at (396.6, 78.0)
- added H1: MountingHole, MountingHole:MountingHole_3.2mm_M3_ISO7380_Pad, F.Cu at (134.0, 69.0)
- added H2: MountingHole, MountingHole:MountingHole_3.2mm_M3_ISO7380_Pad, F.Cu at (166.0, 69.0)
- added H3: MountingHole, MountingHole:MountingHole_3.2mm_M3_ISO7380_Pad, F.Cu at (166.0, 141.0)
- added H4: MountingHole, MountingHole:MountingHole_3.2mm_M3_ISO7380_Pad, F.Cu at (134.0, 141.0)
- added IC2: STM32F730R8T6, ASSETS:QFP50P1200X1200X160-64N, F.Cu at (294.8, 86.6)
- added IC3: ESP32-PICO-V3, ASSETS:ESP32PICOV3, F.Cu at (304.2, 62.4)
- added J10: Conn_01x01, ASSETS:2.54MM PIN, F.Cu at (308.7, 89.1)
- added J11: Conn_01x01, ASSETS:2.54MM PIN, F.Cu at (304.1, 94.7)
- added J12: Conn_01x01, ASSETS:2.54MM PIN, F.Cu at (311.6, 87.2)
- added J13: Conn_01x01, ASSETS:2.54MM PIN, F.Cu at (296.2, 94.6)
- added J14: Conn_01x01, ASSETS:2.54MM PIN, F.Cu at (316.5, 83.6)
- added J15: Conn_01x01, ASSETS:2.54MM PIN, F.Cu at (312.1, 94.0)
- added J16: Conn_01x04, ASSETS:SWD_PINS, F.Cu at (316.0, 80.1)
- added J17: SMA_Edge, ASSETS:SMA-J-P-H-ST-EM1, F.Cu at (157.0, 68.0)
- added J18: SMA_Edge, ASSETS:SMA-J-P-H-ST-EM1, F.Cu at (143.0, 68.0)
- added J19: Conn_01x01, ASSETS:2.54MM PIN, F.Cu at (314.1, 91.1)
- added J20: Conn_01x01, ASSETS:2.54MM PIN, F.Cu at (309.5, 94.0)
- added J21: Conn_01x01, ASSETS:2.54MM PIN, F.Cu at (317.1, 86.5)
- added J3: Conn_01x01, ASSETS:2.54MM PIN, F.Cu at (303.3, 91.8)
- added J4: Conn_01x01, ASSETS:2.54MM PIN, B.Cu at (401.0, 85.6)
- added J5: Conn_01x01, ASSETS:2.54MM PIN, B.Cu at (403.4, 85.6)
- added J6: Conn_01x01, ASSETS:2.54MM PIN, B.Cu at (401.0, 80.4)
- added J7: Conn_01x01, ASSETS:2.54MM PIN, B.Cu at (403.6, 80.5)
- added J8: Conn_01x01, ASSETS:2.54MM PIN, F.Cu at (305.8, 91.8)
- added J9: Conn_01x01, ASSETS:2.54MM PIN, F.Cu at (301.6, 94.7)
- added L1: 2N, Inductor_SMD:L_0402_1005Metric, F.Cu at (313.6, 62.7)
- added L2: L, Inductor_SMD:L_0402_1005Metric, F.Cu at (289.0, 73.6)
- added L3: 15U, Inductor_SMD:L_0402_1005Metric, F.Cu at (156.0, 82.0)
- added L4: 15U, Inductor_SMD:L_0402_1005Metric, F.Cu at (154.4, 81.4)
- added L5: 15U, Inductor_SMD:L_0402_1005Metric, F.Cu at (154.9, 79.9)
- added L6: 15U, Inductor_SMD:L_0402_1005Metric, F.Cu at (158.6, 80.9)
- added L7: 15U, Inductor_SMD:L_0402_1005Metric, F.Cu at (154.9, 76.8)
- added L8: 15U, Inductor_SMD:L_0402_1005Metric, F.Cu at (156.7, 91.6)
- added L9: 15U, Inductor_SMD:L_0402_1005Metric, F.Cu at (156.9, 71.3)
- added R1: R_Small, Resistor_SMD:R_0402_1005Metric, B.Cu at (421.5, 65.1)
- added R10: 100R, Resistor_SMD:R_0402_1005Metric, F.Cu at (314.3, 87.4)
- added R11: 100R, Resistor_SMD:R_0402_1005Metric, F.Cu at (319.2, 83.8)
- added R12: 100R, Resistor_SMD:R_0402_1005Metric, F.Cu at (311.4, 92.3)
- added R13: 100R, Resistor_SMD:R_0402_1005Metric, F.Cu at (314.3, 89.4)
- added R14: 100R, Resistor_SMD:R_0402_1005Metric, F.Cu at (306.8, 96.9)
- added R15: 4.7K, Resistor_SMD:R_0402_1005Metric, F.Cu at (408.5, 114.3)
- added R16: 4.7K, Resistor_SMD:R_0402_1005Metric, F.Cu at (405.6, 114.3)
- added R17: 100R, Resistor_SMD:R_0402_1005Metric, F.Cu at (153.8, 74.5)
- added R18: 100R, Resistor_SMD:R_0402_1005Metric, F.Cu at (160.0, 74.5)
- added R19: 20K, Resistor_SMD:R_0402_1005Metric, F.Cu at (291.9, 75.2)
- added R2: R_Small, Resistor_SMD:R_0402_1005Metric, B.Cu at (404.4, 65.3)
- added R20: 20K, Resistor_SMD:R_0402_1005Metric, F.Cu at (310.4, 74.4)
- added R21: 20K, Resistor_SMD:R_0402_1005Metric, F.Cu at (310.7, 64.7)
- added R22: 100R, Resistor_SMD:R_0402_1005Metric, B.Cu at (389.2, 84.8)
- added R23: 100R, Resistor_SMD:R_0402_1005Metric, B.Cu at (389.2, 82.4)
- added R24: 100R, Resistor_SMD:R_0402_1005Metric, B.Cu at (389.2, 87.8)
- added R25: 100R, Resistor_SMD:R_0402_1005Metric, B.Cu at (398.4, 82.4)
- added R3: R_Small, Resistor_SMD:R_0402_1005Metric, B.Cu at (403.2, 63.1)
- added R4: R_Small, Resistor_SMD:R_0402_1005Metric, B.Cu at (424.4, 65.9)
- added R5: R_Small, Resistor_SMD:R_0402_1005Metric, B.Cu at (405.0, 61.1)
- added R6: R_Small, Resistor_SMD:R_0402_1005Metric, B.Cu at (411.6, 67.1)
- added R7: R_Small, Resistor_SMD:R_0402_1005Metric, B.Cu at (428.6, 67.9)
- added R8: 100R, Resistor_SMD:R_0402_1005Metric, F.Cu at (311.4, 90.3)
- added R9: 100R, Resistor_SMD:R_0402_1005Metric, F.Cu at (306.8, 95.0)
- added U1: W25Q32JVSS, Package_SO:SOIC-8_5.23x5.23mm_P1.27mm, F.Cu at (303.8, 70.8)
- added U2: TXS0108EPW, Package_SO:TSSOP-20_4.4x6.5mm_P0.65mm, F.Cu at (387.4, 120.8)
- added U3: HM01B0, ASSETS:HM01B0, F.Cu at (385.1, 112.1)
- added U4: TXS0108EPW, Package_SO:TSSOP-20_4.4x6.5mm_P0.65mm, F.Cu at (394.6, 120.8)
- added U5: LLCC68_LORA, Package_DFN_QFN:QFN-24-1EP_4x4mm_P0.5mm_EP2.6x2.6mm, F.Cu at (157.0, 87.5)
- added U6: PE4259, ASSETS:SOT65P215X110-6N, F.Cu at (156.8, 75.4)
- added U7: MCP73837T, Package_DFN_QFN:DFN-10-1EP_3x3mm_P0.5mm_EP1.55x2.48mm, B.Cu at (395.6, 85.2)
- added Y1: Crystal_GND23, Crystal:Crystal_SMD_TXC_7M-4Pin_3.2x2.5mm, F.Cu at (311.9, 59.5)
- added Y2: Crystal_GND23, Crystal:Crystal_SMD_SeikoEpson_FA238V-4Pin_3.2x2.5mm, F.Cu at (304.7, 88.7)
- added Y3: Crystal_GND23, Crystal:Crystal_SMD_SeikoEpson_MA406-4Pin_11.7x4.0mm, F.Cu at (308.6, 82.9)
- added Y4: Crystal_GND23, Crystal:Crystal_SMD_SeikoEpson_FA238V-4Pin_3.2x2.5mm, B.Cu at (157.2, 87.7)
- D1: value PMEG1030EJ -> LED; footprint Diode_SMD:D_SOD-323F -> LED_SMD:LED_0402_1005Metric
- IC1: moved to B.Cu
- J1: value USB_SMD_105450-0101 -> Micro_SD_Card; footprint ASSETS:MOLEX_105450-0101 -> Connector_Card:microSD_HC_Wuerth_693072010801
- J2: value Conn_01x04 -> USB_SMD_105450-0101; footprint Connector_PinHeader_2.54mm:PinHeader_1x04_P2.54mm_Horizontal -> ASSETS:MOLEX_105450-0101; moved to B.Cu
- moved IC1 214.1 mm to (394.7, 61.5)
- moved J2 188.4 mm to (377.6, 86.0), turned to 90 degrees
- moved J1 137.5 mm to (333.0, 65.2), turned to 0 degrees
- moved Cin1 127.1 mm to (293.2, 96.8), turned to 0 degrees
- moved F1 126.8 mm to (308.9, 87.4), turned to 0 degrees
- moved D1 118.8 mm to (293.4, 94.8)
- moved D2 109.8 mm to (289.6, 95.3)
Connections:
- Cin1 pad 1: +3V3 -> Net-(Cin1-Pad1)
- D1 pad 1: VDD -> GND
- F1 pad 2: Net-(D1-Pad2) -> Net-(D2-Pad2)
- IC1 pad 6: VDD -> Net-(C10-Pad2)
Routing:
- net Net-(C10-Pad2): track 0.00 -> 31.1 mm
- net VDD: track 26.2 -> 38.4 mm
- net +1V8: track 0.00 -> 10.8 mm, vias 0 -> 5
- net Net-(D2-Pad2): track 9.19 -> 0.00 mm
- net GND: track 9.75 -> 1.79 mm, vias 5 -> 1
- net Net-(IC1-Pad3): track 7.19 -> 0.00 mm
- net RFI_P: track 0.00 -> 6.58 mm
- net RFI_N: track 0.00 -> 6.28 mm
- net Net-(C30-Pad2): track 0.00 -> 6.04 mm, vias 0 -> 1
- net Net-(C29-Pad1): track 0.00 -> 5.84 mm, vias 0 -> 1
- net +2V8: track 0.00 -> 5.49 mm, vias 0 -> 2
- net Net-(U3-Pad3): track 0.00 -> 5.25 mm
- net Net-(U3-Pad12): track 0.00 -> 5.23 mm
- net Net-(U3-Pad13): track 0.00 -> 5.17 mm
- net Net-(U3-Pad5): track 0.00 -> 5.13 mm
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- added copper zone on B.Cu, net GND
- added copper zone on F.Cu, net GND
Other:
- board size 29 x 26 mm -> 40 x 80 mm
- copper layers 2 -> 4

Commit message: Add files via upload
Parts:
- removed C50: 270P, Capacitor_SMD:C_0402_1005Metric
- removed J7: Conn_01x01, ASSETS:2.54MM PIN
- removed R20: 20K, Resistor_SMD:R_0402_1005Metric
- J6: value Conn_01x01 -> Conn_01x02; footprint ASSETS:2.54MM PIN -> Battery:BatteryHolder_Keystone_1042_1x18650
- moved C19 193.6 mm to (127.3, 88.2), turned to 180 degrees
- moved C4 191.9 mm to (127.6, 69.5), turned to 180 degrees
- moved C53 191.8 mm to (128.5, 80.3), turned to 180 degrees
- moved C3 189.0 mm to (127.6, 68.4), turned to 180 degrees
- moved C51 188.8 mm to (127.6, 76.6), turned to 180 degrees
- moved C45 188.5 mm to (130.8, 70.7), turned to 180 degrees
- moved C54 186.9 mm to (127.3, 87.1), turned to 180 degrees
- moved C8 185.7 mm to (127.6, 70.7), turned to 180 degrees
- moved C16 185.4 mm to (128.5, 81.4), turned to 180 degrees
- moved L1 184.7 mm to (129.1, 70.1), turned to 270 degrees
- moved C1 184.3 mm to (129.1, 67.9), turned to 270 degrees
- moved C44 183.4 mm to (132.9, 70.7), turned to 180 degrees
- moved C52 180.9 mm to (135.9, 82.0), turned to 270 degrees
- moved C49 180.5 mm to (136.0, 71.5), turned to 180 degrees
- moved C2 180.3 mm to (130.2, 67.9), turned to 270 degrees
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Connections:
- IC3 pad 45: Net-(IC3-Pad45) -> ESPOSC_IN
Routing:
- net +3V3: track 5.43 -> 33.6 mm, vias 0 -> 2
- net CS: track 0.00 -> 11.7 mm, vias 0 -> 2
- net DO: track 0.00 -> 10.2 mm, vias 0 -> 2
- net Net-(C8-Pad1): track 0.00 -> 9.82 mm
- net WP: track 0.00 -> 9.73 mm
- net ESPOSC_IN: track 0.00 -> 9.48 mm, vias 0 -> 2
- net HOLD: track 0.00 -> 9.10 mm
- net CLK: track 0.00 -> 8.90 mm, vias 0 -> 2
- net DI: track 0.00 -> 8.48 mm, vias 0 -> 2
- net Net-(C47-Pad2): track 0.00 -> 7.23 mm
- net ESPOSC_OUT: track 0.00 -> 6.45 mm
- net Net-(C46-Pad2): track 0.00 -> 5.88 mm
- net /ESP32/UART_RX: track 0.00 -> 4.56 mm
- net Net-(IC3-Pad41): track 0.00 -> 3.98 mm
- net /ESP32/ENABLE: track 0.00 -> 3.70 mm, vias 0 -> 1
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- removed copper zone on B.Cu, net GND
- removed copper zone on F.Cu, net GND
Other:
- board size 40 x 80 mm -> 69 x 92 mm

Commit message: Add files via upload
Parts:
- moved C23 39.1 mm to (186.7, 78.9)
- moved C24 39.1 mm to (186.7, 80.0)
- moved C25 39.1 mm to (188.8, 76.8)
- moved C26 39.1 mm to (186.1, 76.3)
- moved C27 39.1 mm to (189.1, 74.7)
- moved C28 39.1 mm to (192.0, 76.2)
- moved C30 39.1 mm to (189.7, 86.5)
- moved C31 39.1 mm to (187.7, 74.7)
- moved C32 39.1 mm to (190.5, 75.8)
- moved C33 39.1 mm to (191.0, 74.2)
- moved C34 39.1 mm to (186.1, 73.2)
- moved C35 39.1 mm to (186.1, 81.7)
- moved C36 39.1 mm to (187.2, 70.9)
- moved C37 39.1 mm to (191.1, 70.9)
- moved C38 39.1 mm to (189.6, 69.3)
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Routing:
- net ESPOSC_IN: track 9.48 -> 7.92 mm
- net +3V3: track 33.6 -> 32.7 mm
- net ESPOSC_OUT: track 6.45 -> 5.89 mm
Other:
- outline, holes or cut-outs redrawn

Commit message: Add files via upload
Parts:
- added Cin2: 2.2uF, Capacitor_SMD:C_0402_1005Metric, B.Cu at (135.7, 111.9)
- added Cin3: 2.2uF, Capacitor_SMD:C_0402_1005Metric, B.Cu at (151.4, 106.6)
- added Cin4: 2.2uF, Capacitor_SMD:C_0402_1005Metric, F.Cu at (149.8, 101.1)
- added Cin5: 2.2uF, Capacitor_SMD:C_0402_1005Metric, B.Cu at (142.1, 109.6)
- added Cin6: 2.2uF, Capacitor_SMD:C_0402_1005Metric, F.Cu at (149.1, 111.4)
- added Cin7: 2.2uF, Capacitor_SMD:C_0402_1005Metric, B.Cu at (135.6, 99.8)
- added Cin8: 2.2uF, Capacitor_SMD:C_0402_1005Metric, F.Cu at (145.3, 114.5)
- added G***: LOGO, ASSETS:Company_Logo1, F.Cu at (143.3, 121.6)
- added J7: Conn_01x01, ASSETS:2.54MM PIN, F.Cu at (133.5, 136.6)
- D4, D5, D6, J2, R22, R23, R24: moved to F.Cu
- J6: value Conn_01x02 -> Conn_01x01; footprint Battery:BatteryHolder_Keystone_1042_1x18650 -> ASSETS:2.54MM PIN; moved to F.Cu
- moved R7 295.2 mm to (138.9, 124.3), turned to 270 degrees
- moved R4 293.9 mm to (135.2, 118.3), turned to 90 degrees
- moved C7 293.1 mm to (140.2, 122.1), turned to 270 degrees
- moved R1 289.6 mm to (137.2, 120.5), turned to 90 degrees
- moved R6 278.2 mm to (138.9, 122.1), turned to 270 degrees
- moved C9 277.4 mm to (132.7, 122.6), turned to 90 degrees
- moved C10 276.8 mm to (131.6, 123.2), turned to 90 degrees
- moved J5 276.5 mm to (131.4, 135.1)
- moved R5 275.2 mm to (137.3, 125.0), turned to 180 degrees
- moved R3 274.0 mm to (135.2, 120.3), turned to 90 degrees
- moved R2 272.4 mm to (137.2, 118.4), turned to 90 degrees
- moved J4 272.0 mm to (133.5, 135.1)
- moved R25 267.5 mm to (135.6, 132.1), turned to 90 degrees
- moved IC1 266.4 mm to (135.5, 123.2), turned to 180 degrees
- moved U7 261.2 mm to (138.0, 128.5), turned to 180 degrees
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Routing:
- net +3V3: track 32.7 -> 136.7 mm, vias 2 -> 29
- net /LoRa/SCK: track 0.00 -> 80.1 mm, vias 0 -> 4
- net /LoRa/MISO: track 0.00 -> 76.7 mm, vias 0 -> 4
- net +1V8: track 10.8 -> 74.0 mm, vias 5 -> 1
- net GND: track 2.29 -> 57.2 mm, vias 1 -> 24
- net /Camera/D5: track 0.00 -> 46.2 mm, vias 0 -> 2
- net /Camera/D6: track 0.00 -> 45.9 mm, vias 0 -> 2
- net LED3_1: track 0.00 -> 44.1 mm, vias 0 -> 2
- net D+: track 0.00 -> 41.4 mm, vias 0 -> 3
- net /LoRa/MOSI: track 0.00 -> 40.5 mm, vias 0 -> 2
- net LED2_1: track 0.00 -> 39.8 mm, vias 0 -> 2
- net /Camera/D7: track 0.00 -> 39.7 mm, vias 0 -> 2
- net /ESP32/ENABLE: track 3.70 -> 43.2 mm, vias 1 -> 2
- net /Camera/SDA: track 0.00 -> 38.7 mm, vias 0 -> 2
- net /LoRa/RESET: track 0.00 -> 38.5 mm, vias 0 -> 2
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- added copper zone on In2.Cu, net +3V3
- added copper zone on B.Cu, net GND
- added copper zone on F.Cu, net GND
- added copper zone on In1.Cu, net GND
Other:
- board size 69 x 92 mm -> 60 x 87 mm
