File: Schematics/IOTv1.sch (KiCad schematic (older format))
At the start: 33 parts, among them IC1 TPS7A2633DRVR, IC2 STM32F730R8T6, J1 USB_SMD_105450-0101, J2 Conn_01x04, U1 HM01B0

Commit message: Add files via upload
Parts:
- removed C1, C2: 10U, Capacitor_SMD:C_0402_1005Metric, symbol Device:C_Small
- removed C3, C4, C5, C6, C7, Cin1: 2.2uF, Capacitor_SMD:C_0402_1005Metric, symbol Device:C_Small
- removed D1, D2: PMEG1030EJ, Diode_SMD:D_SOD-323F, symbol Diode:PMEG1030EJ
- removed F1: ERB-RD1R00X, Fuse:Fuse_0402_1005Metric, symbol Device:Fuse
- removed IC1: TPS7A2633DRVR, ASSETS:TPS7A2633DRVR, symbol Regular_Use:TPS7A2633DRVR
- removed IC2: STM32F730R8T6, ASSETS:QFP50P1200X1200X160-64N, symbol Regular_Use:STM32F730R8T6
- removed J1: USB_SMD_105450-0101, ASSETS:MOLEX_105450-0101, symbol Regular_Use:USB_SMD_105450-0101
- removed J2: Conn_01x04, Connector_PinHeader_2.54mm:PinHeader_1x04_P2.54mm_Horizontal, symbol Connector_Generic:Conn_01x04
- removed R1, R2, R? (x2): 4.7K, Resistor_SMD:R_0402_1005Metric, symbol Device:R_Small
- removed R3, R4, R5, R? (x4): R_Small, Resistor_SMD:R_0402_1005Metric, symbol Device:R_Small
- removed U1: HM01B0, ASSETS:HM01B0, symbol Regular_Use:HM01B0
- removed U? (x2): TXS0108EPW, Package_SO:TSSOP-20_4.4x6.5mm_P0.65mm, symbol Logic_LevelTranslator:TXS0108EPW
- added J1: Micro_SD_Card, Connector_Card:microSD_HC_Wuerth_693072010801, symbol Connector:Micro_SD_Card
- H1, H2, H3, H4: footprint (none) -> MountingHole:MountingHole_3.2mm_M3_ISO7380_Pad
Connections:
- net labels removed: +1V8, +2V8, BOOT0, D+, D-, D0, D1, D2, D3, D4, D5, D6, D7, HSYNC, INT, LED, MCLK, NRST, OSC32_IN, OSC32_OUT, OSC_IN, OSC_OUT, PA0, PA1, PA10, PA15, PA2, PA3, PA4, PA5, PA6, PA7, PA8, PA9, PB0, PB1, PB10, PB11, PB12, PB13, PB14, PB15, PB2, PB3, PB4, PB5, PB6, PB7, PB8, PB9, PC0, PC1, PC10, PC11, PC12, PC2, PC3, PC4, PC6, PC7, PC8, PC9, PD2, PLCK, SCL, SDA, SWCLK, SWDIO, TRIG, VDD, VSYNC
- wire segments 258 -> 40
- no-connect marks 15 -> 0
Other:
- note added: "LoRa"
- note added: "Microcontroller"
- note added: "POWER"
- note added: "Wi/Fi & BLE"
- moved on the sheet: H1, H2, H3, H4
