File: Schematics/Power.sch (KiCad schematic (older format))
At the start: 29 parts, among them IC1 TPS7A2633DRVR, J2 USB_SMD_105450-0101, J4 Conn_01x01, J5 Conn_01x01, J6 Conn_01x01, J7 Conn_01x01, U7 MCP73837T

Commit message: Add files via upload
Parts:
- removed J6, J7: Conn_01x01, ASSETS:2.54MM PIN, symbol Connector_Generic:Conn_01x01
- added J6: Conn_01x02, Battery:BatteryHolder_Keystone_1042_1x18650, symbol Connector_Generic:Conn_01x02
Connections:
- net GND: now also J6.2 (Pin_2)
- net at C10.2, C9.2, D7.1 (K)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: now also J6.1 (Pin_1)
Changed lines of the file:
@@
 Wire Wire Line
 	6950 3500 6050 3500
-$Comp
-L Connector_Generic:Conn_01x01 J?
-U 1 1 609D3DA0
-P 7200 2950
-AR Path="/5FDBCCB2/609D3DA0" Ref="J?"  Part="1"
-AR Path="/5FCD5242/609D3DA0" Ref="J7"  Part="1"
-F 0 "J7" H 7280 2992 50  0000 L CNN
-F 1 "Conn_01x01" H 7280 2901 50  0000 L CNN
-F 2 "ASSETS:2.54MM PIN" H 7200 2950 50  0001 C CNN
-F 3 "~" H 7200 2950 50  0001 C CNN
-	1    7200 2950
-	0    -1   -1   0
-$EndComp
-$Comp
-L Connector_Generic:Conn_01x01 J?
-U 1 1 609D3DA6
-P 7000 2950
-AR Path="/5FDBCCB2/609D3DA6" Ref="J?"  Part="1"
-AR Path="/5FCD5242/609D3DA6" Ref="J6"  Part="1"
-F 0 "J6" H 7080 2992 50  0000 L CNN
-F 1 "Conn_01x01" H 7080 2901 50  0000 L CNN
-F 2 "ASSETS:2.54MM PIN" H 7000 2950 50  0001 C CNN
-F 3 "~" H 7000 2950 50  0001 C CNN
-	1    7000 2950
-	0    -1   -1   0
-$EndComp
+Connection ~ 6950 3500
 Wire Wire Line
-	6950 3500 7000 3500
-Wire Wire Line
-	7000 3500 7000 3150
-Connection ~ 6950 3500
-$Comp
-L power:GND #PWR?
-U 1 1 609D9979
-P 7200 3150
-AR Path="/609D9979" Ref="#PWR?"  Part="1"
-AR Path="/5FDBCCB2/609D9979" Ref="#PWR?"  Part="1"
-AR Path="/5FCD5242/609D9979" Ref="#PWR0118"  Part="1"
-F 0 "#PWR0118" H 7200 2900 50  0001 C CNN
-F 1 "GND" H 7205 2977 50  0000 C CNN
-F 2 "" H 7200 3150 50  0001 C CNN
-F 3 "" H 7200 3150 50  0001 C CNN
-	1    7200 3150
-	-1   0    0    -1
-$EndComp
-Wire Wire Line
-	7600 3500 7000 3500
+	7600 3500 7150 3500
 Connection ~ 7600 3500
-Connection ~ 7000 3500
 $Comp
 L Diode:PMEG1030EJ D?
@@
 Wire Wire Line
 	4800 5750 4750 5750
+$Comp
+L Connector_Generic:Conn_01x02 J6
+U 1 1 5F90E152
+P 7450 2950
+F 0 "J6" V 7414 2762 50  0000 R CNN
+F 1 "Conn_01x02" V 7323 2762 50  0000 R CNN
+F 2 "Battery:BatteryHolder_Keystone_1042_1x18650" H 7450 2950 50  0001 C CNN
+F 3 "~" H 7450 2950 50  0001 C CNN
+	1    7450 2950
+	0    -1   -1   0
+$EndComp
+Wire Wire Line
+	7450 3150 7450 3400
+Wire Wire Line
+	7450 3400 7150 3400
+Wire Wire Line
+	7150 3400 7150 3500
+Connection ~ 7150 3500
+$Comp
+L power:GND #PWR?
+U 1 1 5F914054
+P 7550 3150
+AR Path="/5F914054" Ref="#PWR?"  Part="1"
+AR Path="/5FDBCCB2/5F914054" Ref="#PWR?"  Part="1"
+AR Path="/5FCD5242/5F914054" Ref="#PWR069"  Part="1"
+F 0 "#PWR069" H 7550 2900 50  0001 C CNN
+F 1 "GND" H 7555 2977 50  0000 C CNN
+F 2 "" H 7550 3150 50  0001 C CNN
+F 3 "" H 7550 3150 50  0001 C CNN
+	1    7550 3150
+	-1   0    0    -1
+$EndComp
+Wire Wire Line
+	6950 3500 7150 3500
 $EndSCHEMATC

Commit message: Add files via upload
Parts:
- removed J6: Conn_01x02, Battery:BatteryHolder_Keystone_1042_1x18650, symbol Connector_Generic:Conn_01x02
- added J6, J7: Conn_01x01, ASSETS:2.54MM PIN, symbol Connector_Generic:Conn_01x01
Connections:
- net GND: now also J7.1 (Pin_1)
- net at C10.2, C9.2, D7.1 (K)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: now also J6.1 (Pin_1)
Changed lines of the file:
@@
 encoding utf-8
 Sheet 2 6
-Title ""
-Date ""
-Rev ""
-Comp ""
+Title "BSE Home Surveillance Node"
+Date "2020-10-19"
+Rev "v1"
+Comp "Blackshield Engineering"
 Comment1 ""
 Comment2 ""
@@
 Wire Wire Line
 	4800 5750 4750 5750
-$Comp
-L Connector_Generic:Conn_01x02 J6
-U 1 1 5F90E152
-P 7450 2950
-F 0 "J6" V 7414 2762 50  0000 R CNN
-F 1 "Conn_01x02" V 7323 2762 50  0000 R CNN
-F 2 "Battery:BatteryHolder_Keystone_1042_1x18650" H 7450 2950 50  0001 C CNN
-F 3 "~" H 7450 2950 50  0001 C CNN
-	1    7450 2950
-	0    -1   -1   0
-$EndComp
 Wire Wire Line
 	7450 3150 7450 3400
@@
 Wire Wire Line
 	6950 3500 7150 3500
+$Comp
+L Connector_Generic:Conn_01x01 J?
+U 1 1 5F949558
+P 7750 3150
+AR Path="/5FDBCCB2/5F949558" Ref="J?"  Part="1"
+AR Path="/5FCD5242/5F949558" Ref="J7"  Part="1"
+F 0 "J7" H 7830 3192 50  0000 L CNN
+F 1 "Conn_01x01" H 7830 3101 50  0000 L CNN
+F 2 "ASSETS:2.54MM PIN" H 7750 3150 50  0001 C CNN
+F 3 "~" H 7750 3150 50  0001 C CNN
+	1    7750 3150
+	1    0    0    -1
+$EndComp
+$Comp
+L Connector_Generic:Conn_01x01 J?
+U 1 1 5F94955E
+P 7250 3150
+AR Path="/5FDBCCB2/5F94955E" Ref="J?"  Part="1"
+AR Path="/5FCD5242/5F94955E" Ref="J6"  Part="1"
+F 0 "J6" H 7330 3192 50  0000 L CNN
+F 1 "Conn_01x01" H 7330 3101 50  0000 L CNN
+F 2 "ASSETS:2.54MM PIN" H 7250 3150 50  0001 C CNN
+F 3 "~" H 7250 3150 50  0001 C CNN
+	1    7250 3150
+	-1   0    0    1
+$EndComp
 $EndSCHEMATC
